Commit message: Add files via upload

File: rover/rover.xacro (robot description, xacro)
@@ -11,5 +11,7 @@
   <!-- ========== GAZEBO MATERIALS ========== -->
   <gazebo reference="base_link">
-    <material>Gazebo/Blue</material>
+    <material>
+      <mesh filename="package://w_rover/meshes/base/color_map.png"/>
+    </material>
   </gazebo>
   <gazebo reference="front_left_wheel">
@@ -33,10 +35,4 @@
     </material>
   </gazebo>
-  <link name="base_footprint"/>
-  <joint name="base_footprint_joint" type="fixed">
-    <parent link="base_footprint"/>
-    <child link="base_link"/>
-    <origin xyz="0 0 0.03" rpy="0 0 0"/>
-  </joint>
   <!-- ========== MAIN BODY ========== -->
   <link name="base_link">
@@ -44,12 +40,11 @@
       <origin xyz="0 0 0.015" rpy="0 0 0"/>
       <geometry>
-        <box size="0.5 0.3 0.03"/>
-      </geometry>
-      <material name="blue"/>
+        <mesh filename="package://w_rover/meshes/base/model.dae" scale="0.5 0.5 0.5"/>
+      </geometry>
     </visual>
     <collision>
       <origin xyz="0 0 0.015" rpy="0 0 0"/>
       <geometry>
-        <box size="0.5 0.3 0.03"/>
+        <mesh filename="package://w_rover/meshes/base/model.dae" scale="0.1 0.1 0.1"/>
       </geometry>
     </collision>
@@ -243,10 +238,11 @@
     <plugin name="left_camera_plugin" filename="libgazebo_ros_camera.so">
       <ros>
-        <namespace>/stereo/left</namespace>
+        <namespace>/left</namespace>
         <remapping>image_raw:=image_raw</remapping>
         <remapping>camera_info:=camera_info</remapping>
       </ros>
-      <camera_name>left_camera</camera_name>
+      <camera_name>left</camera_name>
       <frame_name>camera_left_link</frame_name>
+        <camera_info_url>file:///home/ghada/ros2_ws/calibration/left.yaml</camera_info_url>
     </plugin>
   </sensor>
@@ -271,10 +267,11 @@
     <plugin name="right_camera_plugin" filename="libgazebo_ros_camera.so">
       <ros>
-        <namespace>/stereo/right</namespace>
+        <namespace>/right</namespace>
         <remapping>image_raw:=image_raw</remapping>
         <remapping>camera_info:=camera_info</remapping>
       </ros>
-      <camera_name>right_camera</camera_name>
+      <camera_name>right</camera_name>
       <frame_name>camera_right_link</frame_name>
+        <camera_info_url>file:///home/ghada/ros2_ws/calibration/right.yaml</camera_info_url>
     </plugin>
   </sensor>
@@ -313,4 +310,6 @@
       <ros>
         <namespace>$(arg namespace)</namespace>
+        <remapping>/diff_drive_controller/cmd_vel_unstamped:=/cmd_vel</remapping>
+        <remapping>/diff_drive_controller/odom:=/odom</remapping>
       </ros>
       <parameters>$(find w_rover)/config/rover_controllers.yaml</parameters>
